Commit message: Fixed multiple undetected errors in qube_bringup / first draft of qube_controller

File: src/qube_bringup/urdf/controlled_qube.urdf.xacro (robot description, xacro)
@@ -8,5 +8,5 @@
   <joint name="world_to_base" type="fixed">
     <parent link="world"/>
-    <child link="base"/>
+    <child link="base_link"/>
   </joint>
   <!-- driver argumenter -->
@@ -15,5 +15,5 @@
   <xacro:arg name="simulation" default="false"/>
   <!-- Hent inn qube_driver_ros2_control -->
-  <xacro:include filename="$(find qube_driver)/ros2_control/qube_driver.ros2_control.xacro" />
+  <xacro:include filename="$(find qube_driver)/ros2_control/qube_driver.ros2_control.xacro"/>
   <xacro:qube_driver_ros2_control
     name="qube_driver"

File: src/qube_description/urdf/qube.macro.xacro (robot description, xacro)
@@ -52,5 +52,5 @@
     <xacro:property name="indicator_origo" value="0 0 ${disk_thickness/4}" />
     <!-- Base link -->
-    <link name="base">
+    <link name="base_link">
       <!-- Svart boks -->
       <visual>
@@ -130,5 +130,5 @@
       <origin xyz="0 0 ${base_height/2 + disk_thickness/2}" rpy="0 0 0"/>
       <axis xyz="0 0 1"/>
-      <parent link="base"/>
+      <parent link="base_link"/>
       <child link="disk"/>
     </joint>

File: src/qube_description/urdf/qube.urdf.xacro (robot description, xacro)
@@ -8,5 +8,5 @@
   <joint name="world_to_base" type="fixed">
     <parent link="world"/>
-    <child link="base"/>
+    <child link="base_link"/>
   </joint>
 </robot>

Commit message: fixed controller

File: src/qube_bringup/urdf/controlled_qube.urdf.xacro (robot description, xacro)
@@ -8,5 +8,5 @@
   <joint name="world_to_base" type="fixed">
     <parent link="world"/>
-    <child link="base_link"/>
+    <child link="base"/>
   </joint>
   <!-- driver argumenter -->

File: src/qube_description/urdf/qube.macro.xacro (robot description, xacro)
@@ -49,8 +49,8 @@
     <!-- Indikator -->
     <xacro:property name="indicator_width" value="0.005" />
-    <xacro:property name="indicator_thickness" value="0.002" />
-    <xacro:property name="indicator_origo" value="0 0 ${disk_thickness/4}" />
+    <xacro:property name="indicator_thickness" value="0.004" />
+    <xacro:property name="indicator_origo" value="0 ${disk_radius/2} ${disk_thickness/2}" />
     <!-- Base link -->
-    <link name="base_link">
+    <link name="base">
       <!-- Svart boks -->
       <visual>
@@ -60,20 +60,4 @@
         </geometry>
         <material name="base_black"/>
-      </visual>
-      <!-- Rød stripe top -->
-      <visual>
-        <origin xyz="${stripe1_origo}" rpy="0 0 0"/>
-        <geometry>
-          <box size="${base_xy + 0.005} ${base_xy + 0.005} ${stripe_width}"/>
-        </geometry>
-        <material name="top_stripe_red"/>
-      </visual>
-      <!-- Rød stripe bunn -->
-      <visual>
-        <origin xyz="${stripe2_origo}" rpy="0 0 0"/>
-        <geometry>
-          <box size="${base_xy + 0.005} ${base_xy + 0.005} ${stripe_width}"/>
-        </geometry>
-        <material name="bottom_stripe_red"/>
       </visual>
       <!-- Føtter -->
@@ -107,4 +91,26 @@
       </visual>
     </link>
+    <!-- Top stripe link -->
+    <link name="top_stripe_link">
+      <!-- Rød stripe top -->
+      <visual>
+        <origin xyz="0 0 0" rpy="0 0 0"/>
+        <geometry>
+          <box size="${base_xy + 0.005} ${base_xy + 0.005} ${stripe_width}"/>
+        </geometry>
+        <material name="top_stripe_red"/>
+      </visual>
+    </link>
+    <!-- Bottom stripe link -->
+    <link name="bottom_stripe_link">
+      <!-- Rød stripe bunn -->
+      <visual>
+        <origin xyz="0 0 0" rpy="0 0 0"/>
+        <geometry>
+          <box size="${base_xy + 0.005} ${base_xy + 0.005} ${stripe_width}"/>
+        </geometry>
+        <material name="bottom_stripe_red"/>
+      </visual>
+    </link>
     <!-- Disk link -->
     <link name="disk">
@@ -117,7 +123,10 @@
         <material name="disk_red"/>
       </visual>
+    </link>
+    <!-- Indicator link -->
+    <link name="indicator_link">
       <!-- Hvit indikator -->
       <visual>
-        <origin xyz="${indicator_origo}" rpy="0 0 0"/>
+        <origin xyz="0 0 0" rpy="0 0 0"/>
         <geometry>
           <box size="${indicator_width} ${disk_radius} ${indicator_thickness}"/>
@@ -126,10 +135,28 @@
       </visual>
     </link>
-    <!-- Base til disk : Spinner -->
+    <!-- Fixed joint for top stripe -->
+    <joint name="top_stripe_joint" type="fixed">
+      <origin xyz="${stripe1_origo}" rpy="0 0 0"/>
+      <parent link="base"/>
+      <child link="top_stripe_link"/>
+    </joint>
+    <!-- Fixed joint for bottom stripe -->
+    <joint name="bottom_stripe_joint" type="fixed">
+      <origin xyz="${stripe2_origo}" rpy="0 0 0"/>
+      <parent link="base"/>
+      <child link="bottom_stripe_link"/>
+    </joint>
+    <!-- Base to disk joint -->
     <joint name="motor_joint" type="continuous">
       <origin xyz="0 0 ${base_height/2 + disk_thickness/2}" rpy="0 0 0"/>
       <axis xyz="0 0 1"/>
-      <parent link="base_link"/>
+      <parent link="base"/>
       <child link="disk"/>
+    </joint>
+    <!-- Disk to indicator joint -->
+    <joint name="indicator_joint" type="fixed">
+      <origin xyz="${indicator_origo}" rpy="0 0 0"/>
+      <parent link="disk"/>
+      <child link="indicator_link"/>
     </joint>
   </xacro:macro>

File: src/qube_description/urdf/qube.urdf.xacro (robot description, xacro)
@@ -8,5 +8,5 @@
   <joint name="world_to_base" type="fixed">
     <parent link="world"/>
-    <child link="base_link"/>
+    <child link="base"/>
   </joint>
 </robot>
