Commit message: Ferdig med qube_bringup

File: src/qube_description/urdf/qube.macro.xacro (robot description, xacro)
@@ -127,5 +127,5 @@
     </link>
     <!-- Base til disk : Spinner -->
-    <joint name="disk_joint" type="continuous">
+    <joint name="motor_joint" type="continuous">
       <origin xyz="0 0 ${base_height/2 + disk_thickness/2}" rpy="0 0 0"/>
       <axis xyz="0 0 1"/>

File: src/qube_description/urdf/qube.urdf.xacro (robot description, xacro)
@@ -1,6 +1,8 @@
 <?xml version="1.0"?>
 <robot xmlns:xacro="http://ros.org/wiki/xacro" name="qube">
+  <!-- Hent inn qube modellen -->
   <xacro:include filename="$(find qube_description)/urdf/qube.macro.xacro" />
   <xacro:qube/>
+  <!-- Link Qube til scene -->
   <link name="world"/>
   <joint name="world_to_base" type="fixed">

Commit message: Fikset macro, slettet test

File: src/qube_description/urdf/qube.macro.xacro (robot description, xacro)
@@ -6,6 +6,6 @@
       <color rgba="0 0 0 1"/>
     </material>
-    <material name="top_stripe_red">
-      <color rgba="1 0 0 1"/>
+    <material name="top_stripe_blue">
+      <color rgba="0 0 1 1"/>
     </material>
     <material name="bottom_stripe_red">
@@ -34,5 +34,5 @@
     <xacro:property name="base_height" value="0.112" />
     <!-- Striper -->
-    <xacro:property name="stripe_width" value="0.01" />
+    <xacro:property name="stripe_width" value="0.003" />
     <xacro:property name="stripe1_origo" value="0 0 ${base_height/2 - 0.01}" />
     <xacro:property name="stripe2_origo" value="0 0 ${-(base_height/2 - 0.01)}" />
@@ -48,6 +48,6 @@
     <xacro:property name="disk_thickness" value="0.01" />
     <!-- Indikator -->
-    <xacro:property name="indicator_width" value="0.005" />
-    <xacro:property name="indicator_thickness" value="0.004" />
+    <xacro:property name="indicator_width" value="0.0015" />
+    <xacro:property name="indicator_thickness" value="0.003" />
     <xacro:property name="indicator_origo" value="0 ${disk_radius/2} ${disk_thickness/2}" />
     <!-- Base link -->
@@ -93,11 +93,11 @@
     <!-- Top stripe link -->
     <link name="top_stripe_link">
-      <!-- Rød stripe top -->
+      <!-- Blå stripe top -->
       <visual>
         <origin xyz="0 0 0" rpy="0 0 0"/>
         <geometry>
-          <box size="${base_xy + 0.005} ${base_xy + 0.005} ${stripe_width}"/>
+          <box size="${base_xy + 0.001} ${base_xy + 0.001} ${stripe_width}"/>
         </geometry>
-        <material name="top_stripe_red"/>
+        <material name="top_stripe_blue"/>
       </visual>
     </link>
@@ -108,5 +108,5 @@
         <origin xyz="0 0 0" rpy="0 0 0"/>
         <geometry>
-          <box size="${base_xy + 0.005} ${base_xy + 0.005} ${stripe_width}"/>
+          <box size="${base_xy + 0.001} ${base_xy + 0.001} ${stripe_width}"/>
         </geometry>
         <material name="bottom_stripe_red"/>
@@ -147,12 +147,12 @@
       <child link="bottom_stripe_link"/>
     </joint>
-    <!-- Base to disk joint -->
+    <!-- Base til disk joint -->
     <joint name="motor_joint" type="continuous">
-      <origin xyz="0 0 ${base_height/2 + disk_thickness/2}" rpy="0 0 0"/>
-      <axis xyz="0 0 1"/>
+      <origin xyz="0 0 ${base_height/2 + disk_thickness/2}" rpy="0 0 ${3.1415/4}"/>
+      <axis xyz="0 0 -1"/>
       <parent link="base"/>
       <child link="disk"/>
     </joint>
-    <!-- Disk to indicator joint -->
+    <!-- Disk til indicator joint -->
     <joint name="indicator_joint" type="fixed">
       <origin xyz="${indicator_origo}" rpy="0 0 0"/>
